File: M_Strals_MultiVib/M_Strals_MultiVib.sch (KiCad schematic (older format))
At the start: 0 parts

Commit message: Izveidota jauna komponente un biblioteka. Komponente ievietota shemaa. veikta shemas anotacija un ERC parbaude.
Parts:
- added BT1: 9V, symbol Battery
- added C1, C2: 47uF, symbol CP
- added D1, D2: LED, symbol LED
- added R1, R4: 470R, symbol R
- added R2, R3: 47K, symbol R
- added U1: BC817DS, symbol BC817DS
Connections:
- new net: D1.1 (K), R1.1
- new net: C1.1, R1.2, U1.3 (2_C)
- new net: BT1.1 (+), D1.2 (A), D2.2 (A), R2.1, R3.1
- new net: C1.2, R2.2, U1.2 (1_B)
- new net: C2.2, R3.2, U1.5 (2_B)
- new net: D2.1 (K), R4.1
- new net: C2.1, R4.2, U1.6 (1_C)
- new net: BT1.2 (-), U1.1 (1_E), U1.4 (2_E)
Changed lines of the file:
@@
 LIBS:contrib
 LIBS:valves
+LIBS:bc817ds
+LIBS:M_Strals_MultiVib-cache
 EELAYER 25 0
 EELAYER END
@@
 Comment4 ""
 $EndDescr
+$Comp
+L R R1
+U 1 1 58C11ED7
+P 6100 2650
+F 0 "R1" V 6180 2650 50  0000 C CNN
+F 1 "470R" V 6100 2650 50  0000 C CNN
+F 2 "" V 6030 2650 50  0000 C CNN
+F 3 "" H 6100 2650 50  0000 C CNN
+	1    6100 2650
+	1    0    0    -1
+$EndComp
+$Comp
+L R R2
+U 1 1 58C11F7C
+P 6500 2650
+F 0 "R2" V 6580 2650 50  0000 C CNN
+F 1 "47K" V 6500 2650 50  0000 C CNN
+F 2 "" V 6430 2650 50  0000 C CNN
+F 3 "" H 6500 2650 50  0000 C CNN
+	1    6500 2650
+	1    0    0    -1
+$EndComp
+$Comp
+L R R3
+U 1 1 58C11FD5
+P 6950 2650
+F 0 "R3" V 7030 2650 50  0000 C CNN
+F 1 "47K" V 6950 2650 50  0000 C CNN
+F 2 "" V 6880 2650 50  0000 C CNN
+F 3 "" H 6950 2650 50  0000 C CNN
+	1    6950 2650
+	1    0    0    -1
+$EndComp
+$Comp
+L R R4
+U 1 1 58C12030
+P 7250 2650
+F 0 "R4" V 7330 2650 50  0000 C CNN
+F 1 "470R" V 7250 2650 50  0000 C CNN
+F 2 "" V 7180 2650 50  0000 C CNN
+F 3 "" H 7250 2650 50  0000 C CNN
+	1    7250 2650
+	1    0    0    -1
+$EndComp
+$Comp
+L LED D1
+U 1 1 58C120C5
+P 6100 2100
+F 0 "D1" H 6100 2200 50  0000 C CNN
+F 1 "LED" H 6100 2000 50  0000 C CNN
+F 2 "" H 6100 2100 50  0000 C CNN
+F 3 "" H 6100 2100 50  0000 C CNN
+	1    6100 2100
+	0    -1   -1   0
+$EndComp
+$Comp
+L LED D2
+U 1 1 58C12166
+P 7250 2100
+F 0 "D2" H 7250 2200 50  0000 C CNN
+F 1 "LED" H 7250 2000 50  0000 C CNN
+F 2 "" H 7250 2100 50  0000 C CNN
+F 3 "" H 7250 2100 50  0000 C CNN
+	1    7250 2100
+	0    -1   -1   0
+$EndComp
+$Comp
+L CP C1
+U 1 1 58C121F1
+P 6300 2900
+F 0 "C1" H 6325 3000 50  0000 L CNN
+F 1 "47uF" H 6325 2800 50  0000 L CNN
+F 2 "" H 6338 2750 50  0000 C CNN
+F 3 "" H 6300 2900 50  0000 C CNN
+	1    6300 2900
+	0    -1   -1   0
+$EndComp
+$Comp
+L Battery BT1
+U 1 1 58C1230E
+P 5000 2900
+F 0 "BT1" H 5100 3000 50  0000 L CNN
+F 1 "9V" H 5100 2900 50  0000 L CNN
+F 2 "" V 5000 2960 50  0000 C CNN
+F 3 "" V 5000 2960 50  0000 C CNN
+	1    5000 2900
+	1    0    0    -1
+$EndComp
+$Comp
+L CP C2
+U 1 1 58C124BC
+P 7100 2900
+F 0 "C2" H 7125 3000 50  0000 L CNN
+F 1 "47uF" H 7125 2800 50  0000 L CNN
+F 2 "" H 7138 2750 50  0000 C CNN
+F 3 "" H 7100 2900 50  0000 C CNN
+	1    7100 2900
+	0    1    1    0
+$EndComp
+$Comp
+L BC817DS U1
+U 1 1 58C9B69B
+P 6550 3900
+F 0 "U1" H 6550 4100 60  0000 C CNN
+F 1 "BC817DS" H 6550 4200 60  0000 C CNN
+F 2 "" H 6550 3900 60  0001 C CNN
+F 3 "" H 6550 3900 60  0001 C CNN
+	1    6550 3900
+	1    0    0    -1
+$EndComp
+Wire Wire Line
+	6450 2900 6500 2900
+Wire Wire Line
+	6500 2900 6500 2800
+Connection ~ 6450 2900
+Wire Wire Line
+	6950 2800 6950 3350
+Connection ~ 6950 2900
+Connection ~ 7250 2900
+Connection ~ 6100 2900
+Wire Wire Line
+	7250 2500 7250 2250
+Wire Wire Line
+	6100 2500 6100 2250
+Wire Wire Line
+	5000 1950 7250 1950
+Wire Wire Line
+	5000 1950 5000 2700
+Connection ~ 6100 1950
+Wire Wire Line
+	6500 2500 6500 1950
+Connection ~ 6500 1950
+Wire Wire Line
+	6950 2500 6950 1950
+Connection ~ 6950 1950
+Wire Wire Line
+	6100 3900 6150 3900
+Wire Wire Line
+	6950 4000 6950 4150
+Wire Wire Line
+	6950 4150 5700 4150
+Wire Wire Line
+	5700 4150 5700 3800
+Wire Wire Line
+	5000 3800 6150 3800
+Wire Wire Line
+	6000 2900 6150 2900
+Wire Wire Line
+	5000 3100 5000 3800
+Connection ~ 5700 3800
+Wire Wire Line
+	7250 2800 7250 3800
+Wire Wire Line
+	7250 3800 6950 3800
+Wire Wire Line
+	6100 2900 6100 2800
+Wire Wire Line
+	6000 4000 6150 4000
+Wire Wire Line
+	6950 3350 7000 3350
+Wire Wire Line
+	7000 3350 7000 3900
+Wire Wire Line
+	6450 2900 6450 3400
+Wire Wire Line
+	6450 3400 6100 3400
+Wire Wire Line
+	6100 3400 6100 3900
+Wire Wire Line
+	7000 3900 6950 3900
+Wire Wire Line
+	6000 4000 6000 2900
 $EndSCHEMATC

Commit message: Izveidota shema
Changed lines of the file:
@@
 $Descr A4 11693 8268
 encoding utf-8
-Sheet 1 1
+Sheet 1 2
 Title "M_Strals_MultiVib"
 Date "2017-03-09"
@@
 	5000 1950 7250 1950
 Wire Wire Line
-	5000 1950 5000 2700
+	5000 1600 5000 2700
 Connection ~ 6100 1950
 Wire Wire Line
@@
 Wire Wire Line
 	6000 4000 6000 2900
+$Sheet
+S 8350 2700 900  600
+U 58CA6896
+F0 "Tranzistors" 60
+F1 "Tranzistors.sch" 60
+F2 "Input" I L 8350 2850 60
+F3 "+U" I L 8350 3000 60
+F4 "GND" I L 8350 3150 60
+$EndSheet
+$Comp
+L PWR_FLAG #FLG?
+U 1 1 58CA8155
+P 5000 1600
+F 0 "#FLG?" H 5000 1695 50  0001 C CNN
+F 1 "PWR_FLAG" H 5000 1780 50  0000 C CNN
+F 2 "" H 5000 1600 50  0000 C CNN
+F 3 "" H 5000 1600 50  0000 C CNN
+	1    5000 1600
+	1    0    0    -1
+$EndComp
+Connection ~ 5000 1950
 $EndSCHEMATC
